File: hardware/PWNSAT/USB.kicad_sch (KiCad schematic)
At the start: 51 parts, among them J1 USB_A, J10 Battery, J6 USB_A, P4 USB_C_Plug_USB2.0, Q1 DMG3415U-7, SW1 ON, SW4 USB Selector, U1 FSUSB30MUX, U1 SL2.1A, U2 TP4056, U4 MT3608, U5 AP2114H-3.3, Y5 Crystal_GND2

Commit message: feat(Hw):Init_Floorplan
Parts:
- J3: renamed from J10; footprint Footprints:BatteryHolder_Keystone_1042_1x18650 -> PWNCube:BatteryHolder_Keystone_1042_1x18650
- J4: renamed from J1; footprint Footprints:USB_A_Connfly_DS1095 -> PWNCube:USB_A_Connfly_DS1095
- J5: renamed from J6; footprint Footprints:USB_A_Connfly_DS1095 -> PWNCube:USB_A_Connfly_DS1095
- L5: renamed from L1; footprint Footprints:LQH5BPN -> PWNCube:LQH5BPN
- P1: renamed from P4; footprint Footprints:C393939 -> PWNCube:C393939
- U5: renamed from U1; footprint Footprints:IC_FSUSB42UMX -> PWNCube:IC_FSUSB42UMX
- U8: renamed from U1; footprint Package_SO:SOP-16_3.9x9.9mm_P1.27mm -> Package_SO:SO-16_3.9x9.9mm_P1.27mm
- renumbered C10 to C46, C9 to C47, C18 to C48, C11 to C49, C22 to C50, C21 to C51, C7 to C52, C31 to C53, C32 to C54, C1 to C55, C2 to C56, C8 to C57, D12 to D2, D16 to D3, D8 to D4, D9 to D5, D14 to D6, D15 to D7, F3 to F2, F4 to F3, H4 to H1, H3 to H2, H2 to H3, H1 to H4, R14 to R26, R15 to R27, R13 to R28, R46 to R29, R19 to R30, R44 to R32, R11 to R33, R45 to R34, R32 to R35, R37 to R36, R1 to R37, SW1 to SW3, U2 to U4, U4 to U6, U5 to U7, Y5 to Y3
