File: hardware/PWNSAT/untitled.kicad_sch (KiCad schematic)
At the start: 55 parts, among them J2 Conn_01x04_Pin, SW1 SW_Push, SW2 SW_Push, U2 W25N02KVZEIR, Y1 Crystal, Y2 24MHz

Commit message: feat(Hw):BoM´s_Updated
Parts:
- C14, C15, C18, C2, C24, C26, C30, C6, C7: LCSC# C77020 -> C56392
- C19, C20, C21, C22: Mnfr# GRM1555C2A180GA01D -> (none)
- R2: LCSC# (none) -> C728568
- R6, R8: LCSC# (none) -> C313374
