File: hardware/Sensor_Board/Sensors.kicad_sch (KiCad schematic)
At the start: 29 parts, among them J1 Antenna, U1 ICM-42670-P, U10 PE42421, U12 SX1262IMLTRT, U4 BME280, U9 0900FM15D0039, Y4 32Mhz

Commit message: feat(Hw):Batt_Board_Pro_Added
Parts:
- added C14, C3, C4: 0.1uF, Capacitor_SMD:C_0402_1005Metric, symbol CatSniffer-rescue:C_Small-Device-CatStick-rescue-CatSniffer-rescue
- added C15: 100pF, Capacitor_SMD:C_0402_1005Metric, symbol CatSniffer-rescue:C-Device-CatStick-rescue-CatSniffer-rescue
- added C16, C18: 3.3pF, Capacitor_SMD:C_0402_1005Metric, symbol CatSniffer-rescue:C-Device-CatStick-rescue-CatSniffer-rescue
- added C19, C20: 1nF, Capacitor_SMD:C_0402_1005Metric, symbol CatSniffer-rescue:C_Small-Device-CatStick-rescue-CatSniffer-rescue
- added C5: 47pF, Capacitor_SMD:C_0402_1005Metric, symbol CatSniffer-rescue:C_Small-Device-CatStick-rescue-CatSniffer-rescue
- added C6: 470nF, Capacitor_SMD:C_0402_1005Metric, symbol CatSniffer-rescue:C_Small-Device-CatStick-rescue-CatSniffer-rescue
- added J2: Antenna, FlatSat:SMA_EDGE, symbol CatSniffer-rescue:Conn_Coaxial-Connector-CatStick-rescue-CatSniffer-rescue
- added JP2: Jumper, Jumper:SolderJumper-3_P1.3mm_Bridged12_RoundedPad1.0x1.5mm_NumberLabels, symbol CatSniffer-rescue:Jumper_3_Bridged12-Jumper-CatStick-rescue-CatSniffer-rescue
- added L2: 47nH, Inductor_SMD:L_0603_1608Metric, symbol CatSniffer-rescue:L_Small-Device-CatStick-rescue-CatSniffer-rescue
- added L3: 15uH, Inductor_SMD:L_0603_1608Metric, symbol CatSniffer-rescue:L_Small-Device-CatStick-rescue-CatSniffer-rescue
- added L5: 9.1nH, Inductor_SMD:L_0603_1608Metric, symbol CatSniffer-rescue:L-Device-CatStick-rescue-CatSniffer-rescue
- added R2, R3: 100R, Resistor_SMD:R_0402_1005Metric, symbol CatSniffer-rescue:R_Small-Device-CatStick-rescue-CatSniffer-rescue
- added U2: SX1262IMLTRT, Package_DFN_QFN:QFN-24-1EP_4x4mm_P0.5mm_EP2.65x2.65mm, symbol SX1262IMLTRT:SX1262IMLTRT
- added U3: 0900FM15D0039, FlatSat:0900FM15D0039E, symbol CatSniffer-rescue:0900FM15D0039-Electronic_Cats-CatStick-rescue-CatSniffer-resc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
- added U5: PE42421, Package_TO_SOT_SMD:SOT-363_SC-70-6, symbol CatSniffer-rescue:MASWSS0115-RF_Switch-CatStick-rescue-CatSniffer-rescue
- added Y1: 32Mhz, Crystal:Crystal_SMD_2520-4Pin_2.5x2.0mm, symbol CatSniffer-rescue:Crystal_GND24-Device-CatStick-rescue-CatSniffer-rescue
Connections:
- net +3V3: now also C14.1, C3.1, U2.1 (VDD_IN), U2.10 (VBAT), U2.11 (VBAT_IO)
- net GND: now also C14.2, C16.2, C18.2, C19.2, C20.2, C3.2, C4.2, C5.2, C6.2, J2.2 (Ext), U2.2 (GND), U2.20 (GND), U2.25 (EXP), U2.5 (GND), U2.8 (GND), U3.10 (GND), U3.2 (GND), U3.5 (GND), U3.7 (GND), U3.9 (GND), U5.2 (GND), Y1.2, Y1.4
- new net: C4.1, C5.1, L2.1, U2.24 (VR_PA)
- new net: C16.1, J2.1 (In), L5.1
- new net: C6.1, L3.2, U2.7 (VREG)
- new net: C19.1, R2.1, U5.6 (V1)
- new net: L3.1, U2.9 (DCC_SW)
- new net: C20.1, R3.1, U5.4 (V2)
- new net: C15.2, C18.1, L5.2
- new net: JP2.2 (C), R3.2
- new net: C15.1, U5.5 (RFC)
- new net: U3.8 (SW_RFO), U5.1 (RF1)
- new net: U3.6 (SW_RFI), U5.3 (RF2)
- new net DIO23: JP2.1 (A)
- new net R1_ANT_SW: R2.2
- new net R1_BUSY: U2.14 (BUSY)
- new net R1_DIO1: U2.13 (DIO1)
- new net R1_DIO2: JP2.3 (B), U2.12 (DIO2)
- new net R1_DIO3: U2.6 (DIO3)
- new net R1_MISO: U2.16 (MISO)
- new net R1_MOSI: U2.17 (MOSI)
- new net R1_NSS: U2.19 (NSS)
- new net R1_RFI_N: U2.22 (RFI_N), U3.3 (RFI_N)
- new net R1_RFI_P: U2.21 (RFI_P), U3.4 (RFI_P)
- new net R1_RFO: L2.2, U2.23 (RFO), U3.1 (RFO)
- new net R1_RST: U2.15 (~{NRESET})
- new net R1_SCK: U2.18 (SCK)
- new net R1_XTA: U2.3 (XTA), Y1.3
- new net R1_XTB: U2.4 (XTB), Y1.1
Other:
- moved on the sheet: C1, C10, C11, C12, C13, C17, C2, C21, C22, C31, C43, C7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

Commit message: feat(Hw):floorplans_updated
Parts:
- C8: footprint (none) -> Capacitor_SMD:C_0402_1005Metric
- U1: footprint (none) -> Package_LGA:LGA-14_3x2.5mm_P0.5mm_LayoutBorder3x4y
Other:
- moved on the sheet: C7, C8
Changed lines of the file:
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@@
 	)
 	(junction
+		(at 21.59 30.48)
+		(diameter 0)
+		(color 0 0 0 0)
+	)
+	(junction
 		(at 276.86 55.88)
 		(diameter 0)
@@
 	)
 	(junction
-		(at 20.32 26.67)
+		(at 21.59 26.67)
 		(diameter 0)
 		(color 0 0 0 0)
@@
 	)
 	(junction
-		(at 20.32 30.48)
-		(diameter 0)
-		(color 0 0 0 0)
-	)
-	(junction
 		(at 210.058 85.471)
 		(diameter 0)
@@
 	(wire
 		(pts
-			(xy 25.4 31.75) (xy 25.4 30.48)
+			(xy 26.67 31.75) (xy 26.67 30.48)
 		)
 		(stroke
@@
 	(wire
 		(pts
-			(xy 25.4 30.48) (xy 20.32 30.48)
+			(xy 26.67 30.48) (xy 21.59 30.48)
 		)
 		(stroke
@@
 	(wire
 		(pts
-			(xy 15.24 36.83) (xy 15.24 38.1)
+			(xy 16.51 36.83) (xy 16.51 38.1)
 		)
 		(stroke
@@
 	(wire
 		(pts
-			(xy 15.24 30.48) (xy 15.24 31.75)
+			(xy 16.51 30.48) (xy 16.51 31.75)
 		)
 		(stroke
@@
 	(wire
 		(pts
-			(xy 21.59 38.1) (xy 25.4 38.1)
+			(xy 21.59 38.1) (xy 26.67 38.1)
 		)
 		(stroke
@@
 	(wire
 		(pts
-			(xy 20.32 24.13) (xy 20.32 26.67)
+			(xy 21.59 24.13) (xy 21.59 26.67)
 		)
 		(stroke
@@
 	(wire
 		(pts
-			(xy 20.32 26.67) (xy 20.32 30.48)
+			(xy 21.59 26.67) (xy 21.59 30.48)
 		)
 		(stroke
@@
 	(wire
 		(pts
-			(xy 17.78 26.67) (xy 20.32 26.67)
+			(xy 19.05 26.67) (xy 21.59 26.67)
 		)
 		(stroke
@@
 	(wire
 		(pts
-			(xy 20.32 30.48) (xy 15.24 30.48)
+			(xy 16.51 30.48) (xy 21.59 30.48)
 		)
 		(stroke
@@
 	(wire
 		(pts
-			(xy 25.4 38.1) (xy 25.4 36.83)
+			(xy 26.67 38.1) (xy 26.67 36.83)
 		)
 		(stroke
@@
 	(wire
 		(pts
-			(xy 15.24 38.1) (xy 21.59 38.1)
+			(xy 16.51 38.1) (xy 21.59 38.1)
 		)
 		(stroke
@@
 	(hierarchical_label "+3.3V"
 		(shape input)
-		(at 17.78 26.67 180)
+		(at 19.05 26.67 180)
 		(effects
 			(font
@@
 	(symbol
 		(lib_id "power:+3.3V")
-		(at 20.32 24.13 0)
+		(at 21.59 24.13 0)
 		(unit 1)
 		(exclude_from_sim no)
@@
 		(fields_autoplaced yes)
 		(property "Reference" "#PWR016"
-			(at 20.32 27.94 0)
+			(at 21.59 27.94 0)
 			(effects
 				(font
@@
 		)
 		(property "Value" "+3.3V"
-			(at 20.32 19.05 0)
+			(at 21.59 19.05 0)
 			(effects
 				(font
@@
 		)
 		(property "Footprint" ""
-			(at 20.32 24.13 0)
+			(at 21.59 24.13 0)
 			(effects
 				(font
@@
 		)
 		(property "Datasheet" ""
-			(at 20.32 24.13 0)
+			(at 21.59 24.13 0)
 			(effects
 				(font
@@
 		)
 		(property "Description" "Power symbol creates a global label with name \"+3.3V\""
-			(at 20.32 24.13 0)
+			(at 21.59 24.13 0)
 			(effects
 				(font
@@
 	(symbol
 		(lib_id "Device:C_Small")
-		(at 25.4 34.29 0)
+		(at 26.67 34.29 0)
 		(unit 1)
 		(exclude_from_sim no)
@@
 		(dnp no)
 		(property "Reference" "C8"
-			(at 27.94 33.0262 0)
+			(at 29.21 33.0262 0)
 			(effects
 				(font
@@
 		)
 		(property "Value" "2.2uF"
-			(at 26.162 36.576 0)
+			(at 27.432 36.576 0)
 			(effects
 				(font
@@
 			)
 		)
-		(property "Footprint" ""
-			(at 25.4 34.29 0)
+		(property "Footprint" "Capacitor_SMD:C_0402_1005Metric"
+			(at 26.67 34.29 0)
 			(effects
 				(font
@@
 		)
 		(property "Datasheet" "~"
-			(at 25.4 34.29 0)
+			(at 26.67 34.29 0)
 			(effects
 				(font
@@
 		)
 		(property "Description" "Unpolarized capacitor, small symbol"
-			(at 25.4 34.29 0)
+			(at 26.67 34.29 0)
 			(effects
 				(font
@@
 		)
 		(property "Availability" ""
-			(at 25.4 34.29 0)
+			(at 26.67 34.29 0)
 			(effects
 				(font
@@
 		)
 		(property "Check_prices" ""
-			(at 25.4 34.29 0)
+			(at 26.67 34.29 0)
 			(effects
 				(font
@@
 		)
 		(property "Description_1" ""
-			(at 25.4 34.29 0)
+			(at 26.67 34.29 0)
 			(effects
 				(font
@@
 		)
 		(property "MANUFACTURER" ""
-			(at 25.4 34.29 0)
+			(at 26.67 34.29 0)
 			(effects
 				(font
@@
 		)
 		(property "MF" ""
-			(at 25.4 34.29 0)
+			(at 26.67 34.29 0)
 			(effects
 				(font
@@
 		)
 		(property "MP" ""
-			(at 25.4 34.29 0)
+			(at 26.67 34.29 0)
 			(effects
 				(font
@@
 		)
 		(property "PARTREV" ""
-			(at 25.4 34.29 0)
+			(at 26.67 34.29 0)
 			(effects
 				(font
@@
 		)
 		(property "Package" ""
-			(at 25.4 34.29 0)
+			(at 26.67 34.29 0)
 			(effects
 				(font
@@
 		)
 		(property "Price" ""
-			(at 25.4 34.29 0)
+			(at 26.67 34.29 0)
 			(effects
 				(font
@@
 		)
 		(property "STANDARD" ""
-			(at 25.4 34.29 0)
+			(at 26.67 34.29 0)
 			(effects
 				(font
@@
 		)
 		(property "SnapEDA_Link" ""
-			(at 25.4 34.29 0)
+			(at 26.67 34.29 0)
 			(effects
 				(font
@@
 			)
 		)
-		(property "Footprint" ""
+		(property "Footprint" "Package_LGA:LGA-14_3x2.5mm_P0.5mm_LayoutBorder3x4y"
 			(at 66.04 44.45 0)
 			(effects
@@
 	(symbol
 		(lib_id "Device:C_Small")
-		(at 15.24 34.29 0)
+		(at 16.51 34.29 0)
 		(unit 1)
 		(exclude_from_sim no)
@@
 		(dnp no)
 		(property "Reference" "C7"
-			(at 17.78 33.0262 0)
+			(at 12.192 32.512 0)
 			(effects
 				(font
@@
 		)
 		(property "Value" "100nF"
-			(at 16.002 36.576 0)
+			(at 10.414 36.0618 0)
 			(effects
 				(font
@@
 		)
 		(property "Footprint" "Capacitor_SMD:C_0402_1005Metric"
-			(at 15.24 34.29 0)
+			(at 16.51 34.29 0)
 			(effects
 				(font
@@
 		)
 		(property "Datasheet" "~"
-			(at 15.24 34.29 0)
+			(at 16.51 34.29 0)
 			(effects
 				(font
@@
 		)
 		(property "Description" "Unpolarized capacitor, small symbol"
-			(at 15.24 34.29 0)
+			(at 16.51 34.29 0)
 			(effects
 				(font
@@
 		)
 		(property "Availability" ""
-			(at 15.24 34.29 0)
+			(at 16.51 34.29 0)
 			(effects
 				(font
@@
 		)
 		(property "Check_prices" ""
-			(at 15.24 34.29 0)
+			(at 16.51 34.29 0)
 			(effects
 				(font
@@
 		)
 		(property "Description_1" ""
-			(at 15.24 34.29 0)
+			(at 16.51 34.29 0)
 			(effects
 				(font
@@
 		)
 		(property "LCSC#" "C56392"
-			(at 15.24 34.29 0)
+			(at 16.51 34.29 0)
 			(effects
 				(font
@@
 		)
 		(property "MANUFACTURER" ""
-			(at 15.24 34.29 0)
+			(at 16.51 34.29 0)
 			(effects
 				(font
@@
 		)
 		(property "MF" ""
-			(at 15.24 34.29 0)
+			(at 16.51 34.29 0)
 			(effects
 				(font
@@
 		)
 		(property "MP" ""
-			(at 15.24 34.29 0)
+			(at 16.51 34.29 0)
 			(effects
 				(font
@@
 		)
 		(property "PARTREV" ""
-			(at 15.24 34.29 0)
+			(at 16.51 34.29 0)
 			(effects
 				(font
@@
 		)
 		(property "Package" ""
-			(at 15.24 34.29 0)
+			(at 16.51 34.29 0)
 			(effects
 				(font
@@
 		)
 		(property "Price" ""
-			(at 15.24 34.29 0)
+			(at 16.51 34.29 0)
 			(effects
 				(font
@@
 		)
 		(property "STANDARD" ""
-			(at 15.24 34.29 0)
+			(at 16.51 34.29 0)
 			(effects
 				(font
@@
 		)
 		(property "SnapEDA_Link" ""
-			(at 15.24 34.29 0)
+			(at 16.51 34.29 0)
 			(effects
 				(font
@@
 		)
 		(property "#LCSC" "C56392"
-			(at 15.24 34.29 0)
+			(at 16.51 34.29 0)
 			(effects
 				(font

Commit message: feat(Hw):Update_Route_And_3d_Model_PWNsat_Batt_Board_And_Sensors
Connections:
- net +3V3 is gone; now on net +3.3V: C13.1, C14.1, C3.1, C9.1, U12.1 (VDD_IN), U12.10 (VBAT), U12.11 (VBAT_IO), U2.1 (VDD_IN), U2.10 (VBAT), U2.11 (VBAT_IO)
Other:
- moved on the sheet: C10, C11, C13, C14, C3, C43, L4, L7, U12

Commit message: feat(Hw):Boards_Updated
Pending_Sensors_Board
Changed lines of the file:
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@@
 	)
 	(junction
-		(at 29.21 99.06)
-		(diameter 0)
-		(color 0 0 0 0)
-	)
-	(junction
 		(at 66.04 26.67)
 		(diameter 0)
@@
 	(wire
 		(pts
-			(xy 101.6 105.41) (xy 106.68 105.41)
+			(xy 101.6 105.41) (xy 128.27 105.41)
 		)
 		(stroke
@@
 	(wire
 		(pts
+			(xy 128.27 97.79) (xy 128.27 105.41)
+		)
+		(stroke
+			(width 0)
+			(type default)
+		)
+	)
+	(wire
+		(pts
 			(xy 150.622 167.767) (xy 150.622 174.371)
 		)
@@
 	(wire
 		(pts
-			(xy 21.59 99.06) (xy 29.21 99.06)
-		)
-		(stroke
-			(width 0)
-			(type default)
-		)
-	)
-	(wire
-		(pts
 			(xy 44.45 40.64) (xy 49.53 40.64)
 		)
@@
 		)
 	)
-	(label "CSB"
-		(at 106.68 105.41 0)
-		(effects
-			(font
-				(size 1.27 1.27)
-			)
-			(justify left bottom)
-		)
-	)
 	(label "R1_XTA"
 		(at 158.369 179.451 0)
@@
 		)
 	)
-	(label "CSB"
-		(at 21.59 99.06 180)
-		(effects
-			(font
-				(size 1.27 1.27)
-			)
-			(justify right bottom)
-		)
-	)
 	(label "R0_XTA"
 		(at 161.29 74.93 0)
@@
 					(unit 1)
 				)
+			)
+		)
+	)
+	(symbol
+		(lib_id "power:+3.3V")
+		(at 128.27 97.79 0)
+		(unit 1)
+		(exclude_from_sim no)
+		(in_bom yes)
+		(on_board yes)
+		(dnp no)
+		(fields_autoplaced yes)
+		(property "Reference" "#PWR035"
+			(at 128.27 101.6 0)
+			(effects
+				(font
+					(size 1.27 1.27)
+				)
+				(hide yes)
+			)
+		)
+		(property "Value" "+3.3V"
+			(at 128.27 92.71 0)
+			(effects
+				(font
+					(size 1.27 1.27)
+				)
+			)
+		)
+		(property "Footprint" ""
+			(at 128.27 97.79 0)
+			(effects
+				(font
+					(size 1.27 1.27)
+				)
+				(hide yes)
+			)
+		)
+		(property "Datasheet" ""
+			(at 128.27 97.79 0)
+			(effects
+				(font
+					(size 1.27 1.27)
+				)
+				(hide yes)
+			)
+		)
+		(property "Description" "Power symbol creates a global label with name \"+3.3V\""
+			(at 128.27 97.79 0)
+			(effects
+				(font
+					(size 1.27 1.27)
+				)
+				(hide yes)
+			)
+		)
+		(pin "1"
+		)
+		(instances
+			(project "Sensor_Board"
+				(path "/671dafcd-6579-4545-95ba-aa32d81f1541/f9364cb8-a9bf-45cb-96b8-f5c6300f110d"
+					(reference "#PWR035")
+					(unit 1)
+				)

Commit message: fix(Hw):Tracks_modified
Connections:
- net SCL_ICM is gone; now on net SCL_SENS: U1.13 (AP_SCL_/_AP_SCLK)
- net SDA_ICM is gone; now on net SDA_SENS: U1.14 (AP_SDA_/_AP_SDIO_/AP_SDI)
- net SCL_BME280 renamed SCL_SENS
- net SDA_BME280 renamed SDA_SENS

Commit message: feat(Hw):labels_updated
Parts:
- C10, C13, C14, C3, C4, C9: value 0.1uF -> 100nF
- C12, C19, C20, C21: LCSC# C710873 -> C76947
- C8: LCSC# (none) -> C170151
- L3, L7: LCSC# C57838 -> C2885870
Changed lines of the file:
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@@
 			)
 		)
-		(property "LCSC#" "C710873 "
+		(property "LCSC#" "C76947"
 			(at 349.758 68.199 0)
 			(effects
@@
 			)
 		)
-		(property "Value" "0.1uF"
+		(property "Value" "100nF"
 			(at 58.2168 159.893 0)
 			(effects
@@
 			)
 		)
-		(property "Datasheet" "https://datasheet.lcsc.com/lcsc/2110081230_Sunlord-SDFL1608T150KTF_C57838.pdf"
+		(property "Datasheet" "https://www.lcsc.com/datasheet/C2885870.pdf"
 			(at 214.63 58.42 0)
 			(effects
@@
 			)
 		)
-		(property "LCSC#" "C57838"
+		(property "LCSC#" "C2885870"
 			(at 214.63 58.42 0)
 			(effects
@@
 			)
 		)
-		(property "LCSC#" "C710873 "
+		(property "LCSC#" "C76947"
 			(at 271.272 177.038 0)
 			(effects
@@
 			)
 		)
-		(property "LCSC#" "C710873 "
+		(property "LCSC#" "C76947"
 			(at 258.318 192.659 0)
 			(effects
@@
 			)
 		)
-		(property "Value" "0.1uF"
+		(property "Value" "100nF"
 			(at 157.2768 40.005 0)
 			(effects
@@
 			)
 		)
-		(property "Value" "0.1uF"
+		(property "Value" "100nF"
 			(at 123.825 206.883 0)
 			(effects
@@
 			)
 		)
-		(property "Datasheet" "~"
+		(property "Datasheet" ""
 			(at 69.85 86.36 0)
 			(effects
@@
 			)
 		)
-		(property "Datasheet" "~"
+		(property "Datasheet" ""
 			(at 62.23 86.36 0)
 			(effects
@@
 			)
 		)
+		(property "LCSC#" "C170151"
+			(at 26.67 34.29 0)
+			(effects
+				(font
+					(size 1.27 1.27)
+				)
+				(hide yes)
+			)
+		)
 		(pin "2"
 		)
@@
 			)
 		)
-		(property "Value" "0.1uF"
+		(property "Value" "100nF"
 			(at 105.41 165.1 0)
 			(effects
@@
 			)
 		)
-		(property "Value" "0.1uF"
+		(property "Value" "100nF"
 			(at 222.885 87.503 0)
 			(effects
@@
 			)
 		)
-		(property "LCSC#" "C710873 "
+		(property "LCSC#" "C76947"
 			(at 362.712 52.578 0)
 			(effects
@@
 			)
 		)
-		(property "Value" "0.1uF"
+		(property "Value" "100nF"
 			(at 205.74 45.72 0)
 			(effects
@@
 			)
 		)
-		(property "Datasheet" "~"
+		(property "Datasheet" ""
 			(at 16.51 34.29 0)
 			(effects
@@
 			)
 		)
-		(property "Datasheet" "https://datasheet.lcsc.com/lcsc/2110081230_Sunlord-SDFL1608T150KTF_C57838.pdf"
+		(property "Datasheet" "https://www.lcsc.com/datasheet/C2885870.pdf"
 			(at 111.76 179.07 0)
 			(effects
@@
 			)
 		)
-		(property "LCSC#" "C57838"
+		(property "LCSC#" "C2885870"
 			(at 111.76 179.07 0)
 			(effects
